File: hardware/BREAD_Slice.kicad_pcb (KiCad board)
At the start: 2 copper layers, 70 x 100 mm, 16 parts, among them J1 Conn_01x10_Female, U1 AP63205

Commit message: initial commit post-fork to r2
Parts:
- removed Logo1: Logo_Open_Hardware_Small, Symbol:OSHW-Symbol_6.7x6mm_SilkScreen
- added ?: , , F.Cu at (137.5, 86.3)
- added C5: 47u 25V, Capacitor_SMD:CP_Elec_6.3x7.7, F.Cu at (137.5, 83.6)
- added C6: 0.1u, Capacitor_SMD:C_0805_2012Metric_Pad1.18x1.45mm_HandSolder, F.Cu at (160.7, 98.5)
- added D2: WS2812B_5050, kml-custom:WS2812-5050-4PIN, F.Cu at (173.1, 135.7)
- added G***: LOGO, kml-custom:FAST-Logo-Medium, F.Cu at (130.1, 70.3)
- added Ref**: Val**, kml-custom:OSHW_Logo_8mm, F.Cu at (136.0, 107.8)
- added SW1: SW_DIP_x04, Button_Switch_SMD:SW_DIP_SPSTx04_Slide_9.78x12.34mm_W8.61mm_P2.54mm, F.Cu at (135.1, 95.5)
- A1: footprint Module:Arduino_Nano -> kml-custom:Arduino_Nano_Headers
- C1: value 22uF -> 10u
- D1: value WS2812B_5050 -> 1N4007; footprint SparkFun-LED:WS2812-5050-4PIN -> Diode_SMD:D_SOD-123F
- J1: value Conn_01x10_Female -> Conn_01x10_Socket
- U1: footprint Package_TO_SOT_SMD:TSOT-23-6 -> kml-custom:SOIC_05WU-7_DIO-M
- moved D1 68.8 mm to (131.6, 80.9), turned to 180 degrees
Connections:
- net /ESTOP renamed /slice_template/ESTOP
- A1 pad 10: unconnected-(A1-D7-Pad10) -> /slice_template/D7
- A1 pad 11: unconnected-(A1-D8-Pad11) -> /slice_template/D8
- A1 pad 12: unconnected-(A1-D9-Pad12) -> /slice_template/D9
- A1 pad 13: unconnected-(A1-D10-Pad13) -> /slice_template/D10
- A1 pad 14: unconnected-(A1-D11-Pad14) -> /slice_template/D11/MOSI
- A1 pad 15: unconnected-(A1-D12-Pad15) -> /slice_template/D12/MISO
- A1 pad 16: unconnected-(A1-D13-Pad16) -> /slice_template/D13/SCK
- A1 pad 17: unconnected-(A1-3V3-Pad17) -> /slice_template/3V3
- A1 pad 18: unconnected-(A1-AREF-Pad18) -> /slice_template/AREF
- A1 pad 19: unconnected-(A1-A0-Pad19) -> /slice_template/A0
- A1 pad 20: unconnected-(A1-A1-Pad20) -> /slice_template/A1
- A1 pad 21: unconnected-(A1-A2-Pad21) -> /slice_template/A2
- A1 pad 22: unconnected-(A1-A3-Pad22) -> /slice_template/A3
- A1 pad 23: /I2C_DAT -> /slice_template/I2C_DAT/A4
- A1 pad 24: /I2C_CLK -> /slice_template/I2C_CLK/A5
- A1 pad 25: unconnected-(A1-A6-Pad25) -> /slice_template/A6
- A1 pad 26: unconnected-(A1-A7-Pad26) -> /slice_template/A7
- A1 pad 28: unconnected-(A1-~{RESET}-Pad28) -> /slice_template/~{RESET}
- A1 pad 30: unconnected-(A1-VIN-Pad30) -> /slice_template/VIN
- A1 pad 6: /INT -> /slice_template/SYNC/CAN_{INT}
- A1 pad 7: /SYNC -> /slice_template/INT/CAN_{CS}
- A1 pad 8: /LED -> /slice_template/LED
- A1 pad 9: unconnected-(A1-D6-Pad9) -> /slice_template/D6
- D1 pad 1: +5V -> /slice_template/VIN
- D1 pad 2: unconnected-(D1-DOUT-Pad2) -> +12V
- J1 pad 3: /I2C_CLK -> /slice_template/I2C_CLK
- J1 pad 4: /I2C_DAT -> /slice_template/I2C_DAT
- J1 pad 7: /INT -> /slice_template/SYNC
- J1 pad 8: /SYNC -> /slice_template/INT
Routing:
- net /slice_template/LED: track 0.00 -> 92.9 mm
- net /LED: track 92.9 -> 0.00 mm
- net /I2C_CLK: track 46.3 -> 0.00 mm
- net /I2C_DAT: track 46.0 -> 0.00 mm
- net GND: track 16.8 -> 57.3 mm, vias 20 -> 19
- net /slice_template/VIN: track 0.00 -> 34.6 mm
- net /slice_template/I2C_DAT/A4: track 0.00 -> 31.1 mm
- net /slice_template/I2C_CLK/A5: track 0.00 -> 31.0 mm
- net /SYNC: track 23.7 -> 0.00 mm
- net /INT: track 23.3 -> 0.00 mm
- net /slice_template/INT/CAN_{CS}: track 0.00 -> 15.4 mm
- net /slice_template/SYNC/CAN_{INT}: track 0.00 -> 14.9 mm
- net /slice_template/I2C_CLK: track 0.00 -> 10.2 mm
- net /slice_template/I2C_DAT: track 0.00 -> 10.0 mm
- net /slice_template/INT: track 0.00 -> 6.49 mm
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- removed copper zone on B.Cu, net GNDPWR
